File: Eagle/modEEGamp_v1.1.sch (EAGLE design)
At the start: 111 parts, among them IC201 TLC277P, IC202 INA114P, IC203 INA114P, IC204 TLC277P, IC205 TLC277P, IC206 TLC277P, J201 PINHD-2X17, P201 20k, P202 20k, P203 20k, Q201 BC557, Q202 BC557, Q203 BC557, Q204 BC557, Q205 BC547, Q206 BC547, Q207 BC547, Q208 BC547

Commit message: New version!
Parts:
- removed C201: 47µF tan 1ohm, DISCRETE@3:ELC-2,5
- removed C202: 10nF, DISCRETE:CAPNP-5@2
- removed C203: 10nF, DISCRETE:CAPNP-7,5
- removed C204, C205: 100pF, DISCRETE:CAPNP-7,5
- removed C208: 100nF, DISCRETE:CAPNP-7,5
- removed C209: 10pF, DISCRETE:CAPNP-7,5
- removed C211, C225, C227: 100nF, DISCRETE:CAPNP-5@2
- removed C212, C216, C222, C232: 1nF, DISCRETE:CAPNP-7,5
- removed C213: 47µF, DISCRETE@2:ELC-5
- removed C214, C217: 100nF, DISCRETE:CAPNP-5
- removed C220: 1µF, DISCRETE:CAPNP-7,5@2
- removed C229: 1µF, DISCRETE:CAPNP-7,5@3
- removed C231: 220nF 5%, DISCRETE:CAPNP-5
- removed C234: 33nF 5%, DISCRETE:CAPNP-5
- removed IC201: TLC277P, BURR:OPA2604AP
- removed IC202, IC203: INA114P, BURR:INA114P
- removed IC205, IC206: TLC277P, BURR:TLC277P
- removed J201: PINHD-2X17, pinhead_:PINHD-2X17
- removed P201: 20k, TRIMPOT:S64Y
- removed P202: 20k, TRIMPOT@2:S64Y
- removed PAD201, R_LEG: (no value), WIREPAD:1,6/0,8
- removed PAD203: U_cal, WIREPAD@2:1,6/0,8
- removed PAD204: Cal_GND, WIREPAD@2:1,6/0,8
- removed PAD205: COM, WIREPAD:1,6/0,8
- removed PAD206: AGND, WIREPAD:1,6/0,8
- removed Q201, Q203: BC557, pnp:BC557
- removed Q205, Q207: BC547, NPN:BC547
- removed R201, R202, R205, R206, R207, R208: 2k2, DISCRETE:RESEU-10
- removed R213: 200k, DISCRETE:RESEU-10
- removed R214, R215: 2k2, DISCRETE:RESEU-7,5
- removed R219: 10k, DISCRETE:RESEU-10@2
- removed R220: 1k, DISCRETE:RESEU-7,5
- removed R221, R230: 100k, DISCRETE:RESEU-7,5
- removed R223, R227: 1M, DISCRETE:RESEU-10@2
- removed R224, R231: 1M, DISCRETE:RESEU-7,5
- removed R228: 15k, DISCRETE:RESEU-7,5@2
- removed R229: 8.2k, DISCRETE:RESEU-7,5
- removed R232: 10k, DISCRETE:RESEU-7,5@2
- removed R238, R239: 10k, DISCRETE:RESEU-7,5
- removed R240: 100, DISCRETE:RESEU-7,5
- removed SJ201, SJ202, SJ203, SJ204, SJ205, SJ206: SJ, JUMPER:SJ
- added C1, C17: 220nf, resistor:C-USC1206
- added C10, C9: 1nF, DISCRETE:CAPNP-7,5
- added C11, C2: 1µF, resistor:C-USC1206
- added C12, C13, C14, C18, C19, C20, C21, C22, C23, C24, C25, C26, C27, C28, C3, C4, C8: 100nF, resistor:C-USC1206
- added C15: 33nF 5%, DISCRETE:CAPNP-5
- added C16: 220nF 5%, DISCRETE:CAPNP-5
- added C5, C6: 100pF, resistor:C-USC1206
- added C7: 10pF, resistor:C-USC1206
- added IC1: AD780N, analog-devices:AD780N
- added IC2, IC4: INA217P, burr-brown:INA217P
- added IC3: TLC277P, BURR:TLC277P
- added P1: 20k, TRIMPOT@2:S64Y
- added Q1, Q3: BC547, NPN:BC547
- added Q2, Q4: BC557, pnp:BC557
- added R1: 25k, resistor:R-TRIMM64Y
- added R10, R11, R12, R4, R5, R7, R8, R9: 2k2, resistor:R-US_0207/2V
- added R13, R16: 100k, resistor:R-US_0207/2V
- added R14: 1k, resistor:R-US_0207/2V
- added R15, R18, R2: 1M, resistor:R-US_0207/2V
- added R17: 8.2k, resistor:R-US_0207/2V
- added R19, R6: 10k, resistor:R-US_0207/2V
- added R20: 15k, resistor:R-US_0207/2V
- added R21, R3: 7.5k, resistor:R-US_0207/2V
- added SJ1: (no value), jumper:SJW
- added TPB1A, TPB1B, TPB2A, TPB2B, TPB3A, TPB3B, TPIAB: (no value), WIREPAD:1,6/0,8
- added U$1: AD7902, EEG:AD7902
- added U$16, U$2, U$28, U$29, U$3, U$35: AD8021, EEG:AD8021
- added X1: RJ45-6L-B, con-tycoelectronics:RJ45-6L-B
- C206, C207, C210: device DISCRETE:CAPNP-7,5 -> resistor:C-USC1206
- C215, C218, C219, C226: device DISCRETE:CAPNP-5 -> resistor:C-USC1206
- C221: device DISCRETE:CAPNP-7,5@2 -> resistor:C-USC1206
- C223, C230: device DISCRETE:CAPNP-5@2 -> resistor:C-USC1206
- C228: device DISCRETE:CAPNP-7,5@3 -> resistor:C-USC1206
- R203, R204, R209, R210, R211, R212, R218: device DISCRETE:RESEU-10 -> resistor:R-US_0207/2V
- R216, R217, R222, R225, R226, R234, R235, R236: device DISCRETE:RESEU-7,5 -> resistor:R-US_0207/2V
- R233, R237: device DISCRETE:RESEU-7,5@2 -> resistor:R-US_0207/2V
- renumbered PAD202 to TPIAA
Connections:
- removed net 2.0V: C202.1, IC201A.+IN, J201.2
- removed net PWM: J201.30, R223.2
- removed net R_LEG: C212.1, C216.1, R213.1, R_LEG.P
- removed net VGND: C201.1, C204.2, C205.1, C206.2, C207.1, C208.1, C211.1, C214.2, C215.2, C217.2, C218.2, C219.2, C223.2, C225.2, C226.1, C231.1, C235.1, IC201A.-IN, IC201A.OUT, IC202.REF, IC203.REF, J201.3, P201.1, P202.2, P202.3, P203.2, P203.3, Q201.E, Q202.E, Q203.E, Q204.E, Q205.E, Q206.E, Q207.E, Q208.E, R224.1, R226.1, R229.1, R231.1, R234.1, R236.1, R238.2, R240.1
- new net N$55: C18.1, U$16SUPPLY.+VS
- new net N$56: C19.1, U$3SUPPLY.+VS
- new net N$58: C20.2, U$3SUPPLY.-VS
- new net N$59: C21.2, U$16SUPPLY.-VS
- new net N$60: C8.1, U$35SUPPLY.+VS
- new net N$61: C12.1, U$28SUPPLY.+VS
- new net N$62: C24.1, U$29SUPPLY.+VS
- new net N$63: C25.2, U$35SUPPLY.-VS
- new net N$64: C26.2, U$28SUPPLY.-VS
- new net N$65: C27.2, U$29SUPPLY.-VS
- new net N$66: R218.1, R6.1, X1.1
- new net N$67: U$1.SDO2, X1.6
- new net N$68: U$1.SDI1, X1.5
- new net VDD: C28.1, U$1.VDD1, U$1.VDD2, U$1.VIO1, U$1.VIO2, X1.3
- new net VREF: C13.2, C14.1, C16.1, C206.2, C207.1, C215.2, C218.2, C219.2, C22.1, C226.1, C23.2, C235.1, C3.2, C4.2, C5.1, C6.2, IC2.REF, IC4.REF, P1.2, P1.3, P203.2, P203.3, Q1.E, Q2.E, Q202.E, Q204.E, Q206.E, Q208.E, Q3.E, Q4.E, R15.1, R17.1, R18.1, R226.1, R234.1, R236.1, U$1.IN1-, U$1.IN2-, X1.2
- net +5V/2: now also C12.2, C14.2, C18.2, C19.2, C22.2, C24.2, C3.1, C8.2, IC1.+VIN, IC2.V+, IC3PWR.VCC, IC4.V+, U$16IC.EN, U$28IC.EN, U$29IC.EN, U$2IC.EN, U$35IC.EN, U$3IC.EN, X1.4; no longer C203.1, C211.2, C213.1, C217.1, C227.2, IC201A.V+, IC202.V+, IC203.V+, IC205PWR.VCC, IC206PWR.VCC, J201.1
- net ADIN0: now also TPB3A.P, U$1.IN1+, U$16IC.-, U$16IC.O; no longer C233.2, C236.2, IC206B.OUT, R235.2, SJ201.2, SJ202.2, SJ203.2
- net ADIN1: now also TPB3B.P, U$1.IN2+, U$35IC.-, U$35IC.O; no longer C232.2, C234.2, IC205B.OUT, R230.2, SJ204.2, SJ205.2, SJ206.2
- net AGND: now also C1.1, C13.1, C17.1, C20.1, C21.1, C23.1, C25.1, C26.1, C27.1, C28.2, C4.1, IC1.GND, IC2.V-, IC3PWR.GND, IC4.V-, R1.E, SJ1.1, U$1.GND@1, U$1.GND@2, U$16IC.LREF, U$28IC.LREF, U$29IC.LREF, U$2IC.LREF, U$35IC.LREF, U$3IC.LREF, X1.8; no longer C201.2, C202.2, C203.2, C208.2, C213.2, C214.1, C225.1, C227.1, C230.1, IC201A.V-, IC202.V-, IC203.V-, IC205PWR.GND, IC206PWR.GND, J201.11, J201.13, J201.5, J201.7, J201.9, P201.3, PAD206.P
- net N$1: now also IC1.VOUT, R1.A, U$1.REF1, U$1.REF2; no longer IC202.RG, R214.1
- net N$10: now also C1.2, R3.2, U$16IC.+; no longer Q203.B, Q207.B, R205.2, R206.1
- net N$13: now also IC3A.+IN, R4.2, R5.2; no longer C204.1, C209.1, Q203.C, Q207.C, R201.2, R205.1
- net N$14: now also IC2.RG1; no longer IC203.RG
- net N$15: now also C2.2, IC4.OUT, TPIAB.P; no longer CH2-.P, R202.1
- net N$16: now also IC4.-IN, R7.2; no longer CH2+.P, R201.1
- net N$17: now also IC4.+IN, R10.2; no longer C220.1, IC205A.+IN, R224.2
- net N$18: now also Q1.B, Q2.B, R7.1, R9.2; no longer C222.1, IC205A.-IN, R220.2, R221.1
- net N$19: now also C5.2, C7.2, Q1.C, Q2.C, R8.2, R9.1; no longer P202.1, R220.1
- net N$2: now also R1.S, R2.2; no longer IC202.RG@1, R215.1
- net N$20: now also IC2.RG2; no longer IC203.RG@1
- net N$21: now also IC2.-IN; no longer IC203.-IN
- net N$22: now also Q3.B, Q4.B, R10.1, R12.2; no longer C222.2, C229.1, IC205A.OUT, R221.2
- net N$23: now also C6.1, C7.1, Q3.C, Q4.C, R11.2, R12.1; no longer C229.2, R231.2, R232.1
- net N$24: now also CH2-.P, R8.1; no longer C232.1, IC205B.-IN, R229.2, R230.1
- net N$25: now also IC2.OUT; no longer IC203.OUT
- net N$26: now also CH2+.P, R11.1; no longer J201.4, SJ201.1
- net N$27: now also IC2.+IN; no longer IC203.+IN
- net N$28: now also U$2IC.+; no longer IC206A.+IN
- net N$3: now also IC1.TRIM, R2.1; no longer IC204B.+IN, R214.2, R215.2
- net N$30: now also C2.1, R15.2, U$28IC.+; no longer PAD204.P, R238.1
- net N$31: now also C9.1, R13.1, R14.2, U$28IC.-; no longer J201.6, SJ202.1
- net N$33: now also P1.1, R14.1; no longer C212.2, IC201B.OUT, R213.2
- net N$34: now also C11.1, C9.2, R13.2, TPB1B.P, U$28IC.O; no longer R227.1, R239.2, R240.2
- net N$35: now also IC3A.-IN, IC3A.OUT, R6.2; no longer J201.8, SJ203.1
- net N$36: now also C15.1, R19.2, R20.1; no longer J201.10, SJ204.1
- net N$37: now also C16.2, R20.2, U$29IC.+; no longer J201.12, SJ205.1
- net N$38: now also U$2IC.-; no longer IC206A.-IN
- net N$4: now also U$1.SDI2, U$1.SDO1; no longer C220.2, IC202.OUT, PAD201.P
- net N$41: now also C11.2, R18.2, R19.1; no longer C216.2, IC201B.-IN, PAD205.P, R218.1, R219.1
- net N$42: now also TPB1A.P, U$2IC.O; no longer IC206A.OUT
- net N$44: now also C10.1, R16.1, R17.2, U$29IC.-; no longer J201.14, SJ206.1
- net N$45: now also IC4.RG1, R4.1; no longer IC204B.-IN, IC204B.OUT, R219.2
- net N$46: now also IC4.RG2, R5.1; no longer R223.1, R227.2
- net N$47: now also C10.2, C15.2, R16.2, R21.1, TPB2B.P, U$29IC.O; no longer IC201B.+IN, P201.2
- net N$48: now also C17.2, R21.2, U$35IC.+; no longer PAD203.P, R239.1
- net N$49: now also U$3IC.-; no longer IC206B.-IN
- net N$5: now also C233.2, C236.2, R235.2, R3.1, TPB2A.P, U$3IC.O; no longer IC202.-IN, R207.2
- net N$53: now also C230.1, U$2SUPPLY.+VS; no longer C234.1, R228.1, R232.2
- net N$54: now also C223.2, U$2SUPPLY.-VS; no longer C231.2, IC205B.+IN, R228.2
- net N$57: now also U$3IC.+; no longer IC206B.+IN
- net N$7: now also U$1.SCK1, U$1.SCK2, X1.7; no longer IC202.+IN, R206.2
- net N$8: now also U$1.CNV1, U$1.CNV2; no longer Q201.B, Q205.B, R207.1, R208.2
- net N$9: now also IC1.O/P, SJ1.2; no longer C205.2, C209.2, Q201.C, Q205.C, R202.2, R208.1
Other:
- note removed: "+2V, buffered"
- note removed: "2 channels must be selected on each"
- note removed: "2.0V buf"
- note removed: "250µVpp +/-10%, 0.1 .. 100Hz"
- note removed: "5Vp-p +/-10% => 250µVp-p +/-10%"
- note removed: "Always connect the unused terminals to VGND, or the DRL will not work properly."
- note removed: "Authors: Moritz v. Buttlar, Joerg Hansmann, Andreas R"
- note removed: "DC checkpoint"
- note removed: "DRL design from http://www.biosemi.com/publications/artikel7.htm, fig.3"
- note removed: "Ground plane is VGND"
- note removed: "HF rejection"
- note removed: "If P201 is needed, adjust potentiometer so DRL=0mV (referred to VGND)"
- note removed: "If you only want to use one channel, never let the other channel float."
- note removed: "Important usage instructions for the DRL."
- note removed: "ModularEEG - 2-channel EEG amplifier module"
- note removed: "Only insert IC201 on _one_ board"
- note removed: "P201 is not needed when INA114 instrumentation amplifiers are used."
- note removed: "PWM cal (PB1)"
- note removed: "Right Leg"
- note removed: "Right-leg driver (DRL) notes:"
- note removed: "See http://openeeg.sf.net for more information."
- note removed: "Square wave Calibration Signal"
- note removed: "The 3rd pole is located on the digital board."
- note removed: "The solder-jumpers (SJ201 - SJ206)"
- note removed: "Use SJ201 and SJ204 for the first board."
- note removed: "Vcc analog"
- note removed: "You may replace it with a short wire from pin 2 and pin 1 (VGND)."
- note removed: "board by closing two jumper gaps with"
- note removed: "boards to share the same connector."
- note removed: "mapping. This allows multiple amplifier"
- note removed: "ref. voltage"
- note removed: "right leg driver"
- note removed: "simulates electrode impedance"
- note removed: "solder."
- note removed: "to the right, are used for channel"
- note removed: "u cal"
- note removed: "voltage divider 1:20000"
- note removed: "when _all_ amplifier inputs are shorted to the DRL output (R_LEG)."
- note removed: "when using 2 or 3 amplifier boards"
- moved on the sheet: C224, C236, CH2+, CH2-

Commit message: Added control board
Parts:
- added VREF: (no value), WIREPAD:1,6/0,8
Connections:
- removed net N$68: U$1.SDI1, X1.5
- net +5V/2: now also U$1.SDI1, U$1.VIO1, U$1.VIO2
- net N$8: now also X1.5
- net VDD: no longer U$1.VIO1, U$1.VIO2
- net VREF: now also VREF.P
Changed lines of the file:
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@@
 <?xml version="1.0" encoding="utf-8"?>
 <!DOCTYPE eagle SYSTEM "eagle.dtd">
-<eagle version="7.2.0">
+<eagle version="7.6.0">
 <drawing>
 <settings>
@@
 <part name="U$14" library="SUPPLY2" deviceset="AGND" device=""/>
 <part name="SJ1" library="jumper" deviceset="SJ" device="W"/>
-<part name="SUPPLY2" library="SUPPLY2" deviceset="VDD" device=""/>
 <part name="R3" library="resistor" deviceset="R-US_" device="0207/2V" value="7.5k"/>
 <part name="C1" library="resistor" deviceset="C-US" device="C1206" value="220nf"/>
@@
 <part name="C28" library="resistor" deviceset="C-US" device="C1206" value="100nF"/>
 <part name="U$40" library="SUPPLY2" deviceset="AGND" device=""/>
+<part name="U$41" library="SUPPLY2" deviceset="+5V/2" device=""/>
+<part name="VREF" library="WIREPAD" deviceset="1,6/0,8" device="" value=" "/>
 </parts>
 <sheets>
@@
 <instance part="U$14" gate="G$1" x="375.92" y="109.22"/>
 <instance part="SJ1" gate="1" x="375.92" y="119.38" rot="R90"/>
-<instance part="SUPPLY2" gate="G$1" x="436.88" y="104.14"/>
 <instance part="R3" gate="G$1" x="330.2" y="154.94"/>
 <instance part="C1" gate="G$1" x="335.28" y="147.32" rot="R180"/>
@@
 <instance part="C28" gate="G$1" x="426.72" y="111.76" rot="MR180"/>
 <instance part="U$40" gate="G$1" x="436.88" y="114.3"/>
+<instance part="U$41" gate="G$1" x="436.88" y="104.14"/>
+<instance part="VREF" gate="P" x="27.94" y="106.68"/>
 </instances>
 <busses>
@@
 <pinref part="C215" gate="G$1" pin="2"/>
 <pinref part="IC2" gate="G$1" pin="REF"/>
+<label x="39.116" y="105.918" size="1.778" layer="95"/>
 </segment>
 <segment>
@@
 <wire x1="457.2" y1="96.52" x2="459.74" y2="96.52" width="0.1524" layer="91"/>
 </segment>
+<segment>
+<pinref part="VREF" gate="P" pin="P"/>
+<wire x1="30.48" y1="106.68" x2="38.1" y2="106.68" width="0.1524" layer="91"/>
+</segment>
 </net>
 <net name="N$12" class="0">
@@
 <pinref part="X1" gate="G$1" pin="4"/>
 <wire x1="449.58" y1="91.44" x2="459.74" y2="91.44" width="0.1524" layer="91"/>
+</segment>
+<segment>
+<pinref part="U$1" gate="G$1" pin="VIO1"/>
+<wire x1="434.34" y1="101.6" x2="436.88" y2="101.6" width="0.1524" layer="91"/>
+<wire x1="436.88" y1="101.6" x2="436.88" y2="99.06" width="0.1524" layer="91"/>
+<pinref part="U$1" gate="G$1" pin="VIO2"/>
+<wire x1="436.88" y1="99.06" x2="436.88" y2="88.9" width="0.1524" layer="91"/>
+<wire x1="436.88" y1="88.9" x2="434.34" y2="88.9" width="0.1524" layer="91"/>
+<pinref part="U$1" gate="G$1" pin="SDI1"/>
+<wire x1="434.34" y1="99.06" x2="436.88" y2="99.06" width="0.1524" layer="91"/>
+<junction x="436.88" y="99.06"/>
+<pinref part="U$41" gate="G$1" pin="+5V/2"/>
+<junction x="436.88" y="101.6"/>
 </segment>
 </net>
@@
 </segment>
 <segment>
-<pinref part="U$1" gate="G$1" pin="VIO1"/>
-<wire x1="434.34" y1="101.6" x2="436.88" y2="101.6" width="0.1524" layer="91"/>
-<wire x1="436.88" y1="101.6" x2="436.88" y2="88.9" width="0.1524" layer="91"/>
-<pinref part="U$1" gate="G$1" pin="VIO2"/>
-<wire x1="436.88" y1="88.9" x2="434.34" y2="88.9" width="0.1524" layer="91"/>
-<pinref part="SUPPLY2" gate="G$1" pin="VDD"/>
-<junction x="436.88" y="101.6"/>
-</segment>
-<segment>
 <pinref part="SUPPLY3" gate="G$1" pin="VDD"/>
 <pinref part="X1" gate="G$1" pin="3"/>
@@
 <pinref part="U$1" gate="G$1" pin="CNV1"/>
 <wire x1="434.34" y1="93.98" x2="444.5" y2="93.98" width="0.1524" layer="91"/>
-<wire x1="444.5" y1="93.98" x2="444.5" y2="81.28" width="0.1524" layer="91"/>
+<wire x1="444.5" y1="93.98" x2="444.5" y2="88.9" width="0.1524" layer="91"/>
 <pinref part="U$1" gate="G$1" pin="CNV2"/>
+<wire x1="444.5" y1="88.9" x2="444.5" y2="81.28" width="0.1524" layer="91"/>
 <wire x1="444.5" y1="81.28" x2="434.34" y2="81.28" width="0.1524" layer="91"/>
+<pinref part="X1" gate="G$1" pin="5"/>
+<wire x1="459.74" y1="88.9" x2="444.5" y2="88.9" width="0.1524" layer="91"/>
+<junction x="444.5" y="88.9"/>
 </segment>
 </net>
@@
 </segment>
 </net>
-<net name="N$68" class="0">
-<segment>
-<pinref part="U$1" gate="G$1" pin="SDI1"/>
-<wire x1="434.34" y1="99.06" x2="447.04" y2="99.06" width="0.1524" layer="91"/>
-<wire x1="447.04" y1="99.06" x2="447.04" y2="88.9" width="0.1524" layer="91"/>
-<pinref part="X1" gate="G$1" pin="5"/>
-<wire x1="447.04" y1="88.9" x2="459.74" y2="88.9" width="0.1524" layer="91"/>
-</segment>
-</net>

Commit message: Finished digital board
Parts:
- removed IC1: AD780N, analog-devices:AD780N
- removed SJ1: (no value), jumper:SJW
- added C29, C30: 100nF, resistor:C-USC1206
- added IC5: TLC277P, BURR:TLC277P
- R1: value 25k -> 10k; device resistor:R-TRIMM64Y -> resistor:R-US_0207/2V
- R2: value 1M -> 10k
Connections:
- net VREF renamed VCOM
- removed net VDD: C28.1, U$1.VDD1, U$1.VDD2, X1.3
- new net N$68: C30.1, IC5PWR.VCC
- net +5V/2: now also C30.2, R2.1; no longer IC1.+VIN
- net AGND: now also C29.1, R1.1; no longer IC1.GND, R1.E, SJ1.1
- net N$1: now also X1.3; no longer IC1.VOUT, R1.A
- net N$2: now also C28.1, IC5A.-IN, IC5A.OUT, U$1.VDD1, U$1.VDD2; no longer R1.S, R2.2
- net N$3: now also C29.2, IC5PWR.GND; no longer IC1.TRIM, R2.1
- net N$9: now also IC5A.+IN, R1.2, R2.2; no longer IC1.O/P, SJ1.2
Other:
- moved on the sheet: R2

Commit message: Switched to DB25
Parts:
- removed X1: RJ45-6L-B, con-tycoelectronics:RJ45-6L-B
- added SJ1, SJ10, SJ11, SJ12, SJ2, SJ3, SJ4, SJ5, SJ6, SJ7, SJ8, SJ9: (no value), jumper:SJ
- added X2: (no value), con-subd:F25HPS
Connections:
- removed net N$67: U$1.SDO2, X1.6
- new net N$69: SJ1.2, X2-25.F
- new net N$70: SJ2.2, X2-13.F
- new net N$71: SJ3.2, X2-24.F
- new net N$72: SJ4.2, X2-12.F
- new net N$73: SJ5.2, X2-23.F
- new net N$74: SJ6.2, X2-11.F
- new net N$75: SJ7.2, X2-22.F
- new net N$76: SJ8.2, X2-10.F
- new net N$77: SJ12.2, X2-8.F
- new net N$78: SJ11.2, X2-20.F
- new net N$79: SJ9.2, X2-21.F
- new net N$80: SJ10.2, X2-9.F
- new net N$81: SJ1.1, SJ10.1, SJ11.1, SJ12.1, SJ2.1, SJ3.1, SJ4.1, SJ5.1, SJ6.1, SJ7.1, SJ8.1, SJ9.1
- net +5V/2: now also X2-17.F; no longer X1.4
- net AGND: now also X2-1.F, X2-14.F, X2-16.F, X2-18.F, X2-4.F, X2-6.F; no longer X1.8
- net N$1: now also X2-3.F; no longer X1.3
- net N$66: now also X2-15.F; no longer X1.1
- net N$7: now also X2-7.F; no longer X1.7
- net N$8: now also X2-19.F; no longer X1.5
- net VCOM: now also X2-2.F, X2-5.F; no longer X1.2

Commit message: Finished up chanes to DB25
Parts:
- removed C13, C14, C29, C30: 100nF, resistor:C-USC1206
- removed IC3, IC5: TLC277P, BURR:TLC277P
- removed R1, R2: 10k, resistor:R-US_0207/2V
- removed SJ1, SJ10, SJ11, SJ12, SJ2, SJ3, SJ4, SJ5, SJ6, SJ7, SJ8, SJ9: (no value), jumper:SJ
- added IC1: (no value), v-reg-micrel:MIC5219XX
Connections:
- removed net N$68: C30.1, IC5PWR.VCC
- removed net N$69: SJ1.2, X2-25.F
- removed net N$70: SJ2.2, X2-13.F
- removed net N$71: SJ3.2, X2-24.F
- removed net N$72: SJ4.2, X2-12.F
- removed net N$73: SJ5.2, X2-23.F
- removed net N$74: SJ6.2, X2-11.F
- removed net N$75: SJ7.2, X2-22.F
- removed net N$76: SJ8.2, X2-10.F
- removed net N$77: SJ12.2, X2-8.F
- removed net N$78: SJ11.2, X2-20.F
- removed net N$79: SJ9.2, X2-21.F
- removed net N$80: SJ10.2, X2-9.F
- removed net N$81: SJ1.1, SJ10.1, SJ11.1, SJ12.1, SJ2.1, SJ3.1, SJ4.1, SJ5.1, SJ6.1, SJ7.1, SJ8.1, SJ9.1
- removed net N$9: IC5A.+IN, R1.2, R2.2
- net +5V/2: now also IC1.EN, IC1.IN; no longer C14.2, C30.2, IC3PWR.VCC, R2.1
- net AGND: now also IC1.GND; no longer C13.1, C29.1, IC3PWR.GND, R1.1
- net N$12: now also IC204B.+IN; no longer IC204A.+IN
- net N$13: now also IC204A.+IN; no longer IC3A.+IN
- net N$2: now also IC1.OUT; no longer IC5A.-IN, IC5A.OUT
- net N$3: now also U$1.SDO2, X2-10.F, X2-11.F, X2-12.F, X2-13.F, X2-20.F, X2-21.F, X2-22.F, X2-23.F, X2-24.F, X2-25.F, X2-8.F, X2-9.F; no longer C29.2, IC5PWR.GND
- net N$35: now also IC204A.-IN, IC204A.OUT; no longer IC3A.-IN, IC3A.OUT
- net N$52: now also IC204B.-IN, IC204B.OUT; no longer IC204A.-IN, IC204A.OUT
- net VCOM: no longer C13.2, C14.1
Other:
- moved on the sheet: IC204A
