File: Eagle/modEEGamp_v1.1.sch (EAGLE design)
At the start: 118 parts, among them IC2 INA217P, IC204 TLC277P, IC4 INA217P, P1 20k, P203 20k, Q1 BC547, Q2 BC557, Q202 BC557, Q204 BC557, Q206 BC547, Q208 BC547, Q3 BC547, Q4 BC557

Commit message: Board shrink
Parts:
- removed 2+PWR, 2-PWR: TSW-102-02-S-S-RA, con-samtec:TSW-102-02-S-S-RA
- removed C2+, C2-: DIN42802, modEEG:DIN42802
- removed C26, C27: 100nF, resistor:C-USC1206
- removed IC4: INA217P, burr-brown:INA217P
- removed R21: 7.5k, resistor:R-US_0207/2V
- removed TPB1B, TPB2B, TPB3B, TPIAB: (no value), WIREPAD:1,6/0,8
- removed U$16, U$2, U$28, U$29, U$3, U$35: AD8021, EEG:AD8021
- added 1+PWR1, 1-PWR1: TSW-101-02-S-D-RA, con-samtec:TSW-101-02-S-D-RA
- added C1+1, C1-1: DIN42802, modEEG:DIN42802
- added C13: 33nF 5%, resistor:C-EUC1206
- added C14: 220nF 5%, resistor:C-EUC1206
- added IC3: INA217DW, burr-brown:INA217DW
- added R2: 2k2, resistor:R-US_R1206
- added TPB1A1, TPB2A1, TPB3A1, TPIAA1: (no value), WIREPAD:1,6/0,8
- added U$10, U$12, U$20, U$30, U$31, U$36: AD8021, EEG:AD8021
- 1+PWR, 1-PWR: value TSW-102-02-S-S-RA -> TSW-101-02-S-D-RA; device con-samtec:TSW-102-02-S-S-RA -> con-samtec:TSW-101-02-S-D-RA
- C1, C12, C18, C19, C20, C206, C207, C21, C210, C215, C218, C223, C230, C24, C25, C3, C4, C5, C6, C7, C8: device resistor:C-USC1206 -> resistor:C-EUC1206
- C10, C224, C233, C9: device DISCRETE:CAPNP-7,5 -> resistor:C-EUC1206
- C11, C2, C221, C228: device resistor:C-USC1206 -> resistor:C-EU050-024X044
- C15: value 33nF 5% -> 220nf; device DISCRETE:CAPNP-5 -> resistor:C-EUC1206
- C16: value 220nF 5% -> 100nF; device DISCRETE:CAPNP-5 -> resistor:C-EUC1206
- C17: value 220nf -> 100nF; device resistor:C-USC1206 -> resistor:C-EUC1206
- C235, C236: device DISCRETE:CAPNP-5 -> resistor:C-EUC1206
- IC2: value INA217P -> INA217DW; device burr-brown:INA217P -> burr-brown:INA217DW
- R1, R10, R11, R203, R204, R209, R210, R211, R212, R216, R217, R218, R222, R225, R226, R233, R234, R235, R236, R237, R3, R4, R5, R6, R7, R8, R9: device resistor:R-US_0207/2V -> resistor:R-US_R1206
- R12: value 2k2 -> 100k; device resistor:R-US_0207/2V -> resistor:R-US_R1206
- R13: value 100k -> 1k; device resistor:R-US_0207/2V -> resistor:R-US_R1206
- R14: value 1k -> 1M; device resistor:R-US_0207/2V -> resistor:R-US_R1206
- R15: value 1M -> 100k; device resistor:R-US_0207/2V -> resistor:R-US_R1206
- R16: value 100k -> 8.2k; device resistor:R-US_0207/2V -> resistor:R-US_R1206
- R17: value 8.2k -> 1M; device resistor:R-US_0207/2V -> resistor:R-US_R1206
- R18: value 1M -> 10k; device resistor:R-US_0207/2V -> resistor:R-US_R1206
- R19: value 10k -> 15k; device resistor:R-US_0207/2V -> resistor:R-US_R1206
- R20: value 15k -> 7.5k; device resistor:R-US_0207/2V -> resistor:R-US_R1206
Connections:
- net N$7 renamed SCK
- net N$8 renamed CNV
- removed net N$10: C1.2, R3.2, U$16IC.+
- removed net N$5 (its old number): C233.2, C236.2, R235.2, R3.1, TPB2A.P, U$3IC.O
- removed net N$55: C18.1, U$16SUPPLY.+VS
- removed net N$56: C19.1, U$3SUPPLY.+VS
- removed net N$58: C20.2, U$3SUPPLY.-VS
- removed net N$59: C21.2, U$16SUPPLY.-VS
- removed net N$60: C8.1, U$35SUPPLY.+VS
- removed net N$61: C12.1, U$28SUPPLY.+VS
- removed net N$62: C24.1, U$29SUPPLY.+VS
- removed net N$63: C25.2, U$35SUPPLY.-VS
- removed net N$64: C26.2, U$28SUPPLY.-VS
- removed net N$65: C27.2, U$29SUPPLY.-VS
- net +5V/2: now also 1+PWR1-2.1, 1-PWR1-2.1, C16.2, C17.2, IC3.V+, U$10IC.EN, U$10SUPPLY.+VS, U$12IC.EN, U$12SUPPLY.+VS, U$20IC.EN, U$20SUPPLY.+VS, U$30IC.EN, U$30SUPPLY.+VS, U$31IC.EN, U$31SUPPLY.+VS, U$36IC.EN, U$36SUPPLY.+VS; no longer 2+PWR-2.1, 2-PWR-2.1, C12.2, C24.2, IC4.V+, U$16IC.EN, U$28IC.EN, U$29IC.EN, U$2IC.EN, U$35IC.EN, U$3IC.EN
- net ADIN0: now also U$20IC.-, U$20IC.O; no longer U$16IC.-, U$16IC.O
- net ADIN1: now also TPB3A1.P, U$36IC.-, U$36IC.O; no longer TPB3B.P, U$35IC.-, U$35IC.O
- net AGND: now also 1+PWR1-1.1, 1-PWR1-1.1, C12.1, C24.1, IC3.V-, U$10IC.LREF, U$10SUPPLY.-VS, U$12IC.LREF, U$12SUPPLY.-VS, U$20IC.LREF, U$20SUPPLY.-VS, U$30IC.LREF, U$30SUPPLY.-VS, U$31IC.LREF, U$31SUPPLY.-VS, U$36IC.LREF, U$36SUPPLY.-VS; no longer 2+PWR-1.1, 2-PWR-1.1, C1.1, C17.1, C26.1, C27.1, IC4.V-, U$16IC.LREF, U$28IC.LREF, U$29IC.LREF, U$2IC.LREF, U$35IC.LREF, U$3IC.LREF
- net N$13: now also C233.2, C236.2, R235.2, R3.1, TPB2A.P, U$12IC.O; no longer IC204A.+IN, R4.2, R5.2
- net N$15: now also C1.2, R3.2, U$20IC.+; no longer C2.2, IC4.OUT, TPIAB.P
- net N$16: now also IC204A.+IN, R2.2, R4.2; no longer IC4.-IN, R7.2
- net N$17: now also C2.2, IC3.OUT, TPIAA1.P; no longer IC4.+IN, R10.2
- net N$18: now also IC3.-IN, R5.2; no longer Q1.B, Q2.B, R7.1, R9.2
- net N$19: now also IC3.+IN, R9.2; no longer C5.2, C7.2, Q1.C, Q2.C, R8.2, R9.1
- net N$22: now also Q1.B, Q2.B, R5.1, R8.2; no longer Q3.B, Q4.B, R10.1, R12.2
- net N$23: now also C5.2, C7.2, Q1.C, Q2.C, R7.2, R8.1; no longer C6.1, C7.1, Q3.C, Q4.C, R11.2, R12.1
- net N$24: now also Q3.B, Q4.B, R11.2, R9.1; no longer C2-.P$1, R8.1
- net N$26: now also C6.1, C7.1, Q3.C, Q4.C, R10.2; no longer C2+.P$1
- net N$28: now also U$10IC.+; no longer U$2IC.+
- net N$30: now also C1-1.P$1, R7.1; no longer C2.1, R15.2, U$28IC.+
- net N$31: now also C1+1.P$1, R10.1; no longer C9.1, R13.1, R14.2, U$28IC.-
- net N$33: now also C2.1, R14.2, U$30IC.+; no longer P1.1, R14.1
- net N$34: now also C9.1, R12.1, U$30IC.-; no longer C11.1, C9.2, TPB1B.P, U$28IC.O
- net N$36: now also P1.1, R13.1; no longer C15.1, R19.2, R20.1
- net N$37: now also C11.1, C9.2, R12.2, TPB1A1.P, U$30IC.O; no longer C16.2, R20.2, U$29IC.+
- net N$38: now also U$10IC.-; no longer U$2IC.-
- net N$41: now also C13.1; no longer C11.2
- net N$42: now also U$10IC.O; no longer U$2IC.O
- net N$44: now also C14.2, R19.2, U$31IC.+; no longer C10.1, R16.1, R17.2, U$29IC.-
- net N$45: now also C11.2, R17.2, R18.1; no longer IC4.RG1, R4.1
- net N$46: now also C10.1, R15.1, R16.2, U$31IC.-; no longer IC4.RG2, R5.1
- net N$47: now also IC3.RG1, R2.1; no longer C10.2, C15.2, R16.2, R21.1, TPB2B.P, U$29IC.O
- net N$48: now also IC3.RG2, R4.1; no longer C17.2, R21.2, U$35IC.+
- net N$49: now also U$12IC.-; no longer U$3IC.-
- net N$53: now also C10.2, C13.2, R15.2, R20.1, TPB2A1.P, U$31IC.O; no longer C230.1, U$2SUPPLY.+VS
- net N$54: now also C15.2, R20.2, U$36IC.+; no longer C223.2, U$2SUPPLY.-VS
- net N$57: now also U$12IC.+; no longer U$3IC.+
- net VCOM: now also C1.1, C12.2, C14.1, C15.1, C17.1, C18.1, C19.1, C20.2, C21.2, C223.2, C230.1, C24.2, C25.2, C8.1, IC3.REF, R14.1, R16.1; no longer IC4.REF, R15.1, R18.1
Other:
- note removed: "Channel 2 +"
- note removed: "Channel 2 -"
- moved on the sheet: 1+PWR-1, 1+PWR-2, 1-PWR-1, 1-PWR-2, C1, C11, C12, C17, C18, C19, C2, C20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

Commit message: Changed to DB-15 connector
Parts:
- removed X2: (no value), con-subd:F25HPS
- added X1: (no value), con-subd:M15HPS
Connections:
- net +5V/2: now also X1-12.M; no longer X2-17.F
- net AGND: now also X1-1.M, X1-11.M, X1-13.M, X1-4.M, X1-6.M, X1-9.M; no longer X2-1.F, X2-14.F, X2-16.F, X2-18.F, X2-4.F, X2-6.F
- net CNV: now also X1-14.M; no longer X2-19.F
- net N$1: now also X1-3.M; no longer X2-3.F
- net N$3: now also X1-8.M; no longer X2-10.F, X2-11.F, X2-12.F, X2-13.F, X2-20.F, X2-21.F, X2-22.F, X2-23.F, X2-24.F, X2-25.F, X2-8.F, X2-9.F
- net N$66: now also X1-10.M; no longer X2-15.F
- net SCK: now also X1-7.M; no longer X2-7.F
- net VCOM: now also X1-2.M, X1-5.M; no longer X2-2.F, X2-5.F
Changed lines of the file:
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@@
 <part name="U$43" library="SUPPLY2" deviceset="+5V/2" device=""/>
 <part name="U$44" library="SUPPLY2" deviceset="AGND" device=""/>
-<part name="X2" library="con-subd" deviceset="F25?S" device="HP"/>
 <part name="U$11" library="SUPPLY2" deviceset="AGND" device=""/>
 <part name="IC1" library="v-reg-micrel" deviceset="MIC5219XX" device=""/>
@@
 <part name="U$49" library="SUPPLY2" deviceset="AGND" device=""/>
 <part name="U$50" library="SUPPLY2" deviceset="AGND" device=""/>
+<part name="X1" library="con-subd" deviceset="M15?S" device="HP"/>
 </parts>
 <sheets>
@@
 <instance part="U$43" gate="G$1" x="500.38" y="124.46"/>
 <instance part="U$44" gate="G$1" x="487.68" y="104.14"/>
-<instance part="X2" gate="-1" x="472.44" y="45.72"/>
-<instance part="X2" gate="-2" x="462.28" y="96.52"/>
-<instance part="X2" gate="-3" x="419.1" y="127"/>
-<instance part="X2" gate="-4" x="472.44" y="40.64"/>
-<instance part="X2" gate="-5" x="462.28" y="99.06"/>
-<instance part="X2" gate="-6" x="472.44" y="35.56"/>
-<instance part="X2" gate="-7" x="462.28" y="83.82"/>
-<instance part="X2" gate="-8" x="533.4" y="86.36"/>
-<instance part="X2" gate="-9" x="533.4" y="83.82"/>
-<instance part="X2" gate="-10" x="533.4" y="81.28"/>
-<instance part="X2" gate="-11" x="533.4" y="78.74"/>
-<instance part="X2" gate="-12" x="533.4" y="76.2"/>
-<instance part="X2" gate="-13" x="533.4" y="73.66"/>
-<instance part="X2" gate="-14" x="472.44" y="43.18"/>
-<instance part="X2" gate="-15" x="27.94" y="157.48"/>
-<instance part="X2" gate="-16" x="472.44" y="38.1"/>
-<instance part="X2" gate="-17" x="462.28" y="91.44"/>
-<instance part="X2" gate="-18" x="472.44" y="33.02"/>
-<instance part="X2" gate="-19" x="462.28" y="88.9"/>
-<instance part="X2" gate="-20" x="533.4" y="55.88"/>
-<instance part="X2" gate="-21" x="533.4" y="53.34"/>
-<instance part="X2" gate="-22" x="533.4" y="50.8"/>
-<instance part="X2" gate="-23" x="533.4" y="48.26"/>
-<instance part="X2" gate="-24" x="533.4" y="45.72"/>
-<instance part="X2" gate="-25" x="533.4" y="43.18"/>
 <instance part="U$11" gate="G$1" x="469.9" y="25.4"/>
 <instance part="IC1" gate="G1" x="490.22" y="116.84" rot="MR0"/>
@@
 <instance part="U$49" gate="G$1" x="-31.75" y="88.9"/>
 <instance part="U$50" gate="G$1" x="-29.21" y="109.22"/>
+<instance part="X1" gate="-1" x="472.44" y="63.5"/>
+<instance part="X1" gate="-2" x="462.28" y="93.98"/>
+<instance part="X1" gate="-3" x="419.1" y="124.46"/>
+<instance part="X1" gate="-4" x="472.44" y="58.42"/>
+<instance part="X1" gate="-5" x="462.28" y="101.6"/>
+<instance part="X1" gate="-6" x="472.44" y="55.88"/>
+<instance part="X1" gate="-7" x="462.28" y="81.28"/>
+<instance part="X1" gate="-8" x="462.28" y="76.2"/>
+<instance part="X1" gate="-9" x="472.44" y="60.96"/>
+<instance part="X1" gate="-10" x="22.86" y="160.02"/>
+<instance part="X1" gate="-11" x="472.44" y="53.34"/>
+<instance part="X1" gate="-12" x="454.66" y="93.98" rot="R90"/>
+<instance part="X1" gate="-13" x="472.44" y="50.8"/>
+<instance part="X1" gate="-14" x="462.28" y="86.36"/>
+<instance part="X1" gate="-15" x="543.56" y="48.26"/>
 </instances>
 <busses>
@@
 </segment>
 <segment>
-<pinref part="X2" gate="-1" pin="F"/>
 <pinref part="U$11" gate="G$1" pin="AGND"/>
-<pinref part="X2" gate="-14" pin="F"/>
-<wire x1="469.9" y1="40.64" x2="469.9" y2="43.18" width="0.1524" layer="91"/>
-<wire x1="469.9" y1="43.18" x2="469.9" y2="45.72" width="0.1524" layer="91"/>
-<junction x="469.9" y="43.18"/>
-<pinref part="X2" gate="-4" pin="F"/>
-<junction x="469.9" y="40.64"/>
-<wire x1="469.9" y1="40.64" x2="469.9" y2="38.1" width="0.1524" layer="91"/>
-<pinref part="X2" gate="-16" pin="F"/>
-<wire x1="469.9" y1="38.1" x2="469.9" y2="35.56" width="0.1524" layer="91"/>
-<junction x="469.9" y="38.1"/>
-<pinref part="X2" gate="-18" pin="F"/>
-<wire x1="469.9" y1="35.56" x2="469.9" y2="33.02" width="0.1524" layer="91"/>
-<wire x1="469.9" y1="33.02" x2="469.9" y2="27.94" width="0.1524" layer="91"/>
-<junction x="469.9" y="33.02"/>
-<pinref part="X2" gate="-6" pin="F"/>
-<junction x="469.9" y="35.56"/>
+<pinref part="X1" gate="-1" pin="M"/>
+<wire x1="469.9" y1="63.5" x2="469.9" y2="60.96" width="0.1524" layer="91"/>
+<pinref part="X1" gate="-9" pin="M"/>
+<wire x1="469.9" y1="60.96" x2="469.9" y2="58.42" width="0.1524" layer="91"/>
+<junction x="469.9" y="60.96"/>
+<pinref part="X1" gate="-4" pin="M"/>
+<wire x1="469.9" y1="58.42" x2="469.9" y2="55.88" width="0.1524" layer="91"/>
+<junction x="469.9" y="58.42"/>
+<pinref part="X1" gate="-6" pin="M"/>
+<wire x1="469.9" y1="55.88" x2="469.9" y2="53.34" width="0.1524" layer="91"/>
+<junction x="469.9" y="55.88"/>
+<pinref part="X1" gate="-11" pin="M"/>
+<wire x1="469.9" y1="53.34" x2="469.9" y2="50.8" width="0.1524" layer="91"/>
+<junction x="469.9" y="53.34"/>
+<pinref part="X1" gate="-13" pin="M"/>
+<wire x1="469.9" y1="50.8" x2="469.9" y2="27.94" width="0.1524" layer="91"/>
+<junction x="469.9" y="50.8"/>
 </segment>
 <segment>
@@
 <wire x1="457.2" y1="106.68" x2="457.2" y2="96.52" width="0.1524" layer="91"/>
 <wire x1="457.2" y1="96.52" x2="459.74" y2="96.52" width="0.1524" layer="91"/>
-<pinref part="X2" gate="-2" pin="F"/>
-<pinref part="X2" gate="-5" pin="F"/>
-<wire x1="459.74" y1="99.06" x2="459.74" y2="96.52" width="0.1524" layer="91"/>
 <junction x="459.74" y="96.52"/>
+<pinref part="X1" gate="-2" pin="M"/>
+<wire x1="459.74" y1="93.98" x2="459.74" y2="96.52" width="0.1524" layer="91"/>
+<pinref part="X1" gate="-5" pin="M"/>
+<wire x1="459.74" y1="96.52" x2="459.74" y2="101.6" width="0.1524" layer="91"/>
 </segment>
 <segment>
@@
 <segment>
 <pinref part="U$39" gate="G$1" pin="+5V/2"/>
-<wire x1="449.58" y1="91.44" x2="459.74" y2="91.44" width="0.1524" layer="91"/>
-<pinref part="X2" gate="-17" pin="F"/>
+<wire x1="449.58" y1="91.44" x2="454.66" y2="91.44" width="0.1524" layer="91"/>
+<pinref part="X1" gate="-12" pin="M"/>
+<wire x1="454.66" y1="91.44" x2="459.74" y2="91.44" width="0.1524" layer="91"/>
+<junction x="454.66" y="91.44"/>
 </segment>
 <segment>
@@
 <pinref part="U$1" gate="G$1" pin="REF1"/>
 <wire x1="411.48" y1="109.22" x2="416.56" y2="109.22" width="0.1524" layer="91"/>
-<wire x1="416.56" y1="109.22" x2="416.56" y2="127" width="0.1524" layer="91"/>
+<wire x1="416.56" y1="109.22" x2="416.56" y2="124.46" width="0.1524" layer="91"/>
 <junction x="416.56" y="109.22"/>
-<pinref part="X2" gate="-3" pin="F"/>
+<pinref part="X1" gate="-3" pin="M"/>
 </segment>
 </net>
@@
 <wire x1="441.96" y1="83.82" x2="459.74" y2="83.82" width="0.1524" layer="91"/>
 <junction x="441.96" y="83.82"/>
-<pinref part="X2" gate="-7" pin="F"/>
+<pinref part="X1" gate="-7" pin="M"/>
+<wire x1="459.74" y1="81.28" x2="459.74" y2="83.82" width="0.1524" layer="91"/>
 </segment>
 </net>
@@
 <wire x1="459.74" y1="88.9" x2="444.5" y2="88.9" width="0.1524" layer="91"/>
 <junction x="444.5" y="88.9"/>
-<pinref part="X2" gate="-19" pin="F"/>
+<pinref part="X1" gate="-14" pin="M"/>
+<wire x1="459.74" y1="86.36" x2="459.74" y2="88.9" width="0.1524" layer="91"/>
 </segment>
 </net>
@@
 <segment>
 <pinref part="R218" gate="G$1" pin="1"/>
-<wire x1="20.32" y1="167.64" x2="20.32" y2="157.48" width="0.1524" layer="91"/>
+<wire x1="20.32" y1="167.64" x2="20.32" y2="160.02" width="0.1524" layer="91"/>
 <pinref part="R6" gate="G$1" pin="1"/>
-<wire x1="20.32" y1="157.48" x2="20.32" y2="152.4" width="0.1524" layer="91"/>
-<wire x1="20.32" y1="157.48" x2="25.4" y2="157.48" width="0.1524" layer="91"/>
-<junction x="20.32" y="157.48"/>
-<pinref part="X2" gate="-15" pin="F"/>
+<wire x1="20.32" y1="160.02" x2="20.32" y2="152.4" width="0.1524" layer="91"/>
+<pinref part="X1" gate="-10" pin="M"/>
+<junction x="20.32" y="160.02"/>
 </segment>
 </net>
 <net name="N$3" class="0">
 <segment>
-<pinref part="X2" gate="-8" pin="F"/>
-<pinref part="X2" gate="-9" pin="F"/>
-<wire x1="530.86" y1="86.36" x2="530.86" y2="83.82" width="0.1524" layer="91"/>
-<pinref part="X2" gate="-10" pin="F"/>
-<wire x1="530.86" y1="83.82" x2="530.86" y2="81.28" width="0.1524" layer="91"/>
-<junction x="530.86" y="83.82"/>
-<pinref part="X2" gate="-11" pin="F"/>
-<wire x1="530.86" y1="81.28" x2="530.86" y2="78.74" width="0.1524" layer="91"/>
-<junction x="530.86" y="81.28"/>
-<pinref part="X2" gate="-12" pin="F"/>
-<wire x1="530.86" y1="78.74" x2="530.86" y2="76.2" width="0.1524" layer="91"/>
-<junction x="530.86" y="78.74"/>
-<pinref part="X2" gate="-13" pin="F"/>
-<wire x1="530.86" y1="76.2" x2="530.86" y2="73.66" width="0.1524" layer="91"/>
-<junction x="530.86" y="76.2"/>
-<pinref part="X2" gate="-20" pin="F"/>
-<wire x1="530.86" y1="73.66" x2="530.86" y2="55.88" width="0.1524" layer="91"/>
-<junction x="530.86" y="73.66"/>
-<pinref part="X2" gate="-21" pin="F"/>
-<wire x1="530.86" y1="55.88" x2="530.86" y2="53.34" width="0.1524" layer="91"/>
-<junction x="530.86" y="55.88"/>
-<pinref part="X2" gate="-22" pin="F"/>
-<wire x1="530.86" y1="53.34" x2="530.86" y2="50.8" width="0.1524" layer="91"/>
-<junction x="530.86" y="53.34"/>
-<pinref part="X2" gate="-23" pin="F"/>
-<wire x1="530.86" y1="50.8" x2="530.86" y2="48.26" width="0.1524" layer="91"/>
-<junction x="530.86" y="50.8"/>
-<pinref part="X2" gate="-24" pin="F"/>
-<wire x1="530.86" y1="48.26" x2="530.86" y2="45.72" width="0.1524" layer="91"/>
-<junction x="530.86" y="48.26"/>
-<pinref part="X2" gate="-25" pin="F"/>
-<wire x1="530.86" y1="45.72" x2="530.86" y2="43.18" width="0.1524" layer="91"/>
-<junction x="530.86" y="45.72"/>
 <pinref part="U$1" gate="G$1" pin="SDO2"/>
-<wire x1="434.34" y1="78.74" x2="530.86" y2="78.74" width="0.1524" layer="91"/>
+<wire x1="434.34" y1="78.74" x2="459.74" y2="78.74" width="0.1524" layer="91"/>
+<pinref part="X1" gate="-8" pin="M"/>
+<wire x1="459.74" y1="76.2" x2="459.74" y2="78.74" width="0.1524" layer="91"/>
 </segment>
 </net>
