File: Eagle/modEEGamp_v1.1.sch (EAGLE design)
At the start: 118 parts, among them IC2 INA217DW, IC204 TLC277P, IC3 INA217DW, P1 20k, P203 20k, Q1 BC547, Q2 BC557, Q202 BC557, Q204 BC557, Q206 BC547, Q208 BC547, Q3 BC547, Q4 BC557

Commit message: Board updates (jumpers)
Parts:
- removed P1, P203: 20k, TRIMPOT@2:S64Y
- added JP1, JP10, JP11, JP12, JP2, JP3, JP4, JP5, JP6, JP7, JP8, JP9: (no value), jumper:JP1Q
- added R21, R22: 20k, resistor:R-TRIMM3296W
- IC1: value (none) -> 2.5V
Connections:
- new net N$10: JP1.2, X2-8.F
- new net N$11: JP2.2, X2-9.F
- new net N$55: JP5.2, X2-12.F
- new net N$56: JP6.2, X2-13.F
- new net N$58: JP7.2, X2-20.F
- new net N$59: JP8.2, X2-21.F
- new net N$6: R13.1, R22.A
- new net N$60: JP9.2, X2-22.F
- new net N$61: JP10.2, X2-23.F
- new net N$62: JP11.2, X2-24.F
- new net N$63: JP12.2, X2-25.F
- new net N$8: R21.A, R222.1
- net N$3: now also JP1.1, JP10.1, JP11.1, JP12.1, JP2.1, JP3.1, JP4.1, JP5.1, JP6.1, JP7.1, JP8.1, JP9.1; no longer X2-10.F, X2-11.F, X2-12.F, X2-13.F, X2-20.F, X2-21.F, X2-22.F, X2-23.F, X2-24.F, X2-25.F, X2-8.F, X2-9.F
- net N$36: now also JP3.2, X2-10.F; no longer P1.1, R13.1
- net N$40: now also JP4.2, X2-11.F; no longer P203.1, R222.1
- net VCOM: now also R21.E, R21.S, R22.E, R22.S; no longer P1.2, P1.3, P203.2, P203.3

Commit message: Part numbers
Parts:
- C1+, C1+1, C1-, C1-1: PN (none) -> Plastics1 41828
Changed lines of the file:
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@@
 <part name="C20" library="resistor" deviceset="C-EU" device="C1206" value="100nF"/>
 <part name="C21" library="resistor" deviceset="C-EU" device="C1206" value="100nF"/>
-<part name="C1-" library="modEEG" deviceset="DIN42802" device=""/>
-<part name="C1+" library="modEEG" deviceset="DIN42802" device=""/>
+<part name="C1-" library="modEEG" deviceset="DIN42802" device="">
+<attribute name="PN" value="Plastics1 41828"/>
+</part>
+<part name="C1+" library="modEEG" deviceset="DIN42802" device="">
+<attribute name="PN" value="Plastics1 41828"/>
+</part>
 <part name="1-PWR" library="con-samtec" deviceset="TSW-101-02-S-D" device="-RA"/>
 <part name="1+PWR" library="con-samtec" deviceset="TSW-101-02-S-D" device="-RA"/>
@@
 <part name="C24" library="resistor" deviceset="C-EU" device="C1206" value="100nF"/>
 <part name="C25" library="resistor" deviceset="C-EU" device="C1206" value="100nF"/>
-<part name="C1-1" library="modEEG" deviceset="DIN42802" device=""/>
-<part name="C1+1" library="modEEG" deviceset="DIN42802" device=""/>
+<part name="C1-1" library="modEEG" deviceset="DIN42802" device="">
+<attribute name="PN" value="Plastics1 41828"/>
+</part>
+<part name="C1+1" library="modEEG" deviceset="DIN42802" device="">
+<attribute name="PN" value="Plastics1 41828"/>
+</part>
 <part name="1-PWR1" library="con-samtec" deviceset="TSW-101-02-S-D" device="-RA"/>
 <part name="1+PWR1" library="con-samtec" deviceset="TSW-101-02-S-D" device="-RA"/>
@@
 <attribute name="VALUE" x="185.42" y="165.1" size="1.778" layer="96" rot="MR180"/>
 </instance>
-<instance part="C1-" gate="G$1" x="-27.94" y="236.22" rot="R180"/>
-<instance part="C1+" gate="G$1" x="-27.94" y="200.66" rot="R180"/>
+<instance part="C1-" gate="G$1" x="-27.94" y="236.22" rot="R180">
+<attribute name="PN" x="-27.94" y="236.22" size="1.778" layer="96" rot="R180" display="off"/>
+</instance>
+<instance part="C1+" gate="G$1" x="-27.94" y="200.66" rot="R180">
+<attribute name="PN" x="-27.94" y="200.66" size="1.778" layer="96" rot="R180" display="off"/>
+</instance>
 <instance part="1-PWR" gate="-1" x="-34.29" y="228.6" rot="R180"/>
 <instance part="1-PWR" gate="-2" x="-34.29" y="231.14" rot="R180"/>
@@
 <attribute name="VALUE" x="182.88" y="48.26" size="1.778" layer="96" rot="MR180"/>
 </instance>
-<instance part="C1-1" gate="G$1" x="-30.48" y="119.38" rot="R180"/>
-<instance part="C1+1" gate="G$1" x="-30.48" y="83.82" rot="R180"/>
+<instance part="C1-1" gate="G$1" x="-30.48" y="119.38" rot="R180">
+<attribute name="PN" x="-30.48" y="119.38" size="1.778" layer="96" rot="R180" display="off"/>
+</instance>
+<instance part="C1+1" gate="G$1" x="-30.48" y="83.82" rot="R180">
+<attribute name="PN" x="-30.48" y="83.82" size="1.778" layer="96" rot="R180" display="off"/>
+</instance>
 <instance part="1-PWR1" gate="-1" x="-36.83" y="111.76" rot="R180"/>
 <instance part="1-PWR1" gate="-2" x="-36.83" y="114.3" rot="R180"/>
