File: Eagle/digital.sch (EAGLE design)
At the start: 53 parts, among them IC1 MAX232, J1 USB+SHIELD

Commit message: Added RTS
Connections:
- new net N$3: IC1G$1.R2IN, X2.7
- new net N$4: IC1G$1.R2OUT, U$1.RC2
Other:
- moved on the sheet: C16, IC1P, OK1A, OK1B, OK2A, OK2B, OK3A, OK3B, OK4A, OK4B, R1, R2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

Commit message: Added connection monitor
Parts:
- added R17, R18: 100k, resistor:R-US_0204/2V
Connections:
- new net N$42: J1.VBUS, R17.1, R18.2
- new net N$55: R17.2, U$1.RA0
- net DGND: now also R18.1
Changed lines of the file:
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@@
 <part name="X2" library="con-subd" deviceset="F09" device="HP"/>
 <part name="SUPPLY60" library="supply2" deviceset="DGND" device=""/>
+<part name="R17" library="resistor" deviceset="R-US_" device="0204/2V" value="100k"/>
+<part name="R18" library="resistor" deviceset="R-US_" device="0204/2V" value="100k"/>
+<part name="SUPPLY4" library="supply2" deviceset="DGND" device=""/>
 </parts>
 <sheets>
@@
 <instance part="X2" gate="G$1" x="233.68" y="17.78"/>
 <instance part="SUPPLY60" gate="G$1" x="226.06" y="10.16"/>
+<instance part="R17" gate="G$1" x="-7.62" y="68.58" rot="R90"/>
+<instance part="R18" gate="G$1" x="-7.62" y="58.42" rot="R90"/>
+<instance part="SUPPLY4" gate="G$1" x="-7.62" y="50.8"/>
 </instances>
 <busses>
@@
 <pinref part="X2" gate="G$1" pin="5"/>
 <pinref part="SUPPLY60" gate="G$1" pin="DGND"/>
+</segment>
+<segment>
+<pinref part="R18" gate="G$1" pin="1"/>
+<pinref part="SUPPLY4" gate="G$1" pin="DGND"/>
 </segment>
 </net>
@@
 </segment>
 </net>
+<net name="N$42" class="0">
+<segment>
+<pinref part="J1" gate="G$1" pin="VBUS"/>
+<wire x1="68.58" y1="2.54" x2="63.5" y2="2.54" width="0.1524" layer="91"/>
+<wire x1="63.5" y1="2.54" x2="63.5" y2="-20.32" width="0.1524" layer="91"/>
+<wire x1="63.5" y1="-20.32" x2="-17.78" y2="-20.32" width="0.1524" layer="91"/>
+<wire x1="-17.78" y1="-20.32" x2="-17.78" y2="63.5" width="0.1524" layer="91"/>
+<pinref part="R17" gate="G$1" pin="1"/>
+<pinref part="R18" gate="G$1" pin="2"/>
+<wire x1="-17.78" y1="63.5" x2="-7.62" y2="63.5" width="0.1524" layer="91"/>
+<junction x="-7.62" y="63.5"/>
+</segment>
+</net>
+<net name="N$55" class="0">
+<segment>
+<pinref part="R17" gate="G$1" pin="2"/>
+<pinref part="U$1" gate="G$1" pin="RA0"/>
+<wire x1="-7.62" y1="73.66" x2="15.24" y2="73.66" width="0.1524" layer="91"/>
+<wire x1="15.24" y1="73.66" x2="15.24" y2="76.2" width="0.1524" layer="91"/>
+</segment>
+</net>
