File: Eagle/modEEGamp_v1.1 - Single.brd (EAGLE design)
At the start: 78.1 x 22.9 mm, 52 parts, among them IC2 INA217DW, P203 20k, Q202 BC557, Q204 BC557, Q206 BC547, Q208 BC547

Commit message: Packages
Parts:
- removed IC2: INA217DW, burr-brown:DW_RPDSO-G16
- added U$1: INA217, modEEG:DIL-08
Connections:
- removed net N$14: IC2.2, R216.1
- removed net N$20: IC2.15, R217.1
- new net N$1: R216.1, U$1.1
- new net N$2: R217.1, U$1.8
- net +5V/2: now also U$1.7; no longer IC2.13
- net AGND: now also U$1.4; no longer IC2.7
- net N$21: now also U$1.2; no longer IC2.4
- net N$25: now also U$1.6; no longer IC2.11
- net N$27: now also U$1.3; no longer IC2.5
- net VCOM: now also U$1.5; no longer IC2.10
Routing:
- net N$14: track 3.59 -> 0.00 mm, vias 1 -> 0
- net N$20: track 3.59 -> 0.00 mm, vias 1 -> 0
- net N$1: track 0.00 -> 3.27 mm
- net N$2: track 0.00 -> 3.27 mm
- net +5V/2: track 123.3 -> 125.3 mm, vias 2 -> 1
- net N$25: track 5.25 -> 7.03 mm
- net N$21: track 3.24 -> 5.01 mm
- net AGND: track 153.3 -> 151.7 mm, vias 10 -> 9
- net N$27: track 3.24 -> 4.49 mm
Changed lines of the file:
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@@
 <element name="C235" library="resistor" package="C1206" value="220nF 5%" x="55.88" y="59.69" rot="R270"/>
 <element name="C236" library="resistor" package="C1206" value="33nF 5%" x="62.23" y="53.34"/>
-<element name="IC2" library="burr-brown" package="DW_RPDSO-G16" value="INA217DW" x="34.29" y="52.07" rot="R270">
-<attribute name="OC_NEWARK" value="02E2758" x="34.29" y="52.07" size="1.778" layer="27" rot="R270" display="off"/>
-<attribute name="MPN" value="INA217AIDWT" x="34.29" y="52.07" size="1.778" layer="27" rot="R270" display="off"/>
-<attribute name="MF" value="TEXAS INSTRUMENTS" x="34.29" y="52.07" size="1.778" layer="27" rot="R270" display="off"/>
-<attribute name="OC_FARNELL" value="1459470" x="34.29" y="52.07" size="1.778" layer="27" rot="R270" display="off"/>
-</element>
 <element name="P203" library="TRIMPOT@2" package="S64Y" value="20k" x="48.26" y="46.355" rot="R90"/>
 <element name="TPIAA" library="WIREPAD" package="1,6/0,8" value=" " x="41.91" y="46.99"/>
@@
 <attribute name="OC_NEWARK" value="unknown" x="2.54" y="50.165" size="1.778" layer="27" rot="R270" display="off"/>
 </element>
+<element name="U$1" library="modEEG" package="DIL-08" value="INA217" x="34.29" y="53.34" rot="R270"/>
 </elements>
 <signals>
 <signal name="AGND">
 <contactref element="C215" pad="1"/>
-<contactref element="IC2" pad="7"/>
 <contactref element="U$2" pad="1"/>
 <contactref element="U$3" pad="1"/>
@@
 <wire x1="9.525" y1="62.865" x2="4.064" y2="57.404" width="0.4064" layer="16"/>
 <wire x1="4.064" y1="53.975" x2="4.064" y2="57.404" width="0.4064" layer="16"/>
-<wire x1="29.49" y1="48.895" x2="31.115" y2="48.895" width="0.4064" layer="1"/>
-<via x="31.115" y="48.895" extent="1-16" drill="0.5"/>
-<wire x1="31.115" y1="48.895" x2="32.89" y2="48.895" width="0.4064" layer="16"/>
 <wire x1="32.89" y1="48.895" x2="33.02" y2="49.025" width="0.4064" layer="16"/>
-<wire x1="31.115" y1="48.895" x2="29.21" y2="50.8" width="0.4064" layer="16"/>
-<wire x1="29.21" y1="50.8" x2="29.21" y2="62.865" width="0.4064" layer="16"/>
 <contactref element="U$16" pad="4"/>
 <contactref element="U$2" pad="4"/>
@@
 <wire x1="43.815" y1="56.515" x2="45.66" y2="56.515" width="0.4064" layer="1"/>
 <wire x1="42.545" y1="62.865" x2="42.545" y2="60.96" width="0.4064" layer="16"/>
-<wire x1="42.545" y1="59.69" x2="42.545" y2="57.785" width="0.4064" layer="16"/>
+<wire x1="42.545" y1="60.96" x2="42.545" y2="57.785" width="0.4064" layer="16"/>
 <wire x1="42.545" y1="57.785" x2="43.815" y2="56.515" width="0.4064" layer="16"/>
 <wire x1="59.63" y1="59.055" x2="59.63" y2="60.9" width="0.4064" layer="1"/>
@@
 <wire x1="42.675" y1="61.09" x2="42.545" y2="60.96" width="0.4064" layer="1"/>
 <via x="42.545" y="60.96" extent="1-16" drill="0.5"/>
-<wire x1="42.545" y1="60.96" x2="42.545" y2="59.69" width="0.4064" layer="16"/>
+<contactref element="U$1" pad="4"/>
+<wire x1="32.89" y1="48.895" x2="31.115" y2="48.895" width="0.4064" layer="16"/>
+<wire x1="31.115" y1="48.895" x2="30.48" y2="49.53" width="0.4064" layer="16"/>
+<wire x1="30.48" y1="49.53" x2="29.21" y2="50.8" width="0.4064" layer="16"/>
+<wire x1="29.21" y1="50.8" x2="29.21" y2="62.865" width="0.4064" layer="16"/>
 </signal>
 <signal name="VCOM">
 <contactref element="C218" pad="2"/>
 <contactref element="C215" pad="2"/>
-<contactref element="IC2" pad="10"/>
 <contactref element="R226" pad="1"/>
 <contactref element="R236" pad="1"/>
@@
 <vertex x="0" y="63.5"/>
 <vertex x="0" y="40.64"/>
-<vertex x="86.36" y="40.64"/>
-<vertex x="86.36" y="63.5"/>
+<vertex x="87.63" y="40.64"/>
+<vertex x="87.63" y="63.5"/>
 </polygon>
 <polygon width="0.4064" layer="1" isolate="0.254">
 <vertex x="0" y="63.5"/>
 <vertex x="0" y="40.64"/>
-<vertex x="82.55" y="40.64"/>
-<vertex x="82.55" y="63.5"/>
+<vertex x="83.82" y="40.64"/>
+<vertex x="83.82" y="63.5"/>
 </polygon>
 <wire x1="53.34" y1="61.09" x2="55.88" y2="61.09" width="0.4064" layer="1"/>
@@
 <via x="55.88" y="43.18" extent="1-16" drill="0.5"/>
 <via x="58.42" y="50.8" extent="1-16" drill="0.5"/>
+<contactref element="U$1" pad="5"/>
 </signal>
 <signal name="N$12">
@@
 <signal name="+5V/2">
 <contactref element="C218" pad="1"/>
-<contactref element="IC2" pad="13"/>
 <contactref element="U$2" pad="8"/>
 <contactref element="U$3" pad="8"/>
@@
 <wire x1="10.16" y1="60.96" x2="6.604" y2="57.404" width="0.4064" layer="16"/>
 <wire x1="6.604" y1="53.975" x2="6.604" y2="57.404" width="0.4064" layer="16"/>
-<wire x1="39.0902" y1="52.705" x2="37.465" y2="52.705" width="0.4064" layer="1"/>
-<via x="37.465" y="52.705" extent="1-16" drill="0.5"/>
-<wire x1="37.465" y1="52.705" x2="37.465" y2="50.93" width="0.4064" layer="16"/>
-<wire x1="37.465" y1="50.93" x2="35.56" y2="49.025" width="0.4064" layer="16"/>
-<wire x1="37.465" y1="52.705" x2="36.195" y2="52.705" width="0.4064" layer="1"/>
-<wire x1="36.195" y1="52.705" x2="35.56" y2="53.34" width="0.4064" layer="1"/>
-<wire x1="35.56" y1="53.34" x2="35.56" y2="62.865" width="0.4064" layer="1"/>
 <contactref element="U$16" pad="7"/>
 <contactref element="U$2" pad="7"/>
@@
 <wire x1="70.99" y1="59.69" x2="70.99" y2="62.735" width="0.4064" layer="1"/>
 <wire x1="70.99" y1="62.735" x2="71.12" y2="62.865" width="0.4064" layer="1"/>
+<contactref element="U$1" pad="7"/>
+<wire x1="38.1" y1="54.61" x2="36.83" y2="54.61" width="0.4064" layer="1"/>
+<wire x1="36.83" y1="54.61" x2="35.56" y2="55.88" width="0.4064" layer="1"/>
+<wire x1="35.56" y1="55.88" x2="35.56" y2="62.865" width="0.4064" layer="1"/>
+<wire x1="35.56" y1="49.025" x2="35.56" y2="49.53" width="0.4064" layer="16"/>
+<wire x1="35.56" y1="49.53" x2="36.83" y2="50.8" width="0.4064" layer="16"/>
+<wire x1="36.83" y1="50.8" x2="38.735" y2="50.8" width="0.4064" layer="16"/>
+<wire x1="38.735" y1="50.8" x2="40.005" y2="52.07" width="0.4064" layer="16"/>
+<wire x1="40.005" y1="52.07" x2="40.005" y2="53.34" width="0.4064" layer="16"/>
+<wire x1="40.005" y1="53.34" x2="38.735" y2="54.61" width="0.4064" layer="16"/>
+<wire x1="38.735" y1="54.61" x2="38.1" y2="54.61" width="0.4064" layer="16"/>
 </signal>
 <signal name="N$25">
 <contactref element="C221" pad="2"/>
 <contactref element="TPIAA" pad="1"/>
-<contactref element="IC2" pad="11"/>
 <wire x1="41.91" y1="46.99" x2="41.91" y2="48.895" width="0.4064" layer="1"/>
-<wire x1="39.09" y1="50.165" x2="40.64" y2="50.165" width="0.4064" layer="1"/>
-<wire x1="40.64" y1="50.165" x2="41.91" y2="48.895" width="0.4064" layer="1"/>
+<contactref element="U$1" pad="6"/>
+<wire x1="38.1" y1="52.07" x2="38.735" y2="52.07" width="0.4064" layer="1"/>
+<wire x1="38.735" y1="52.07" x2="41.91" y2="48.895" width="0.4064" layer="1"/>
 </signal>
 <signal name="ADIN0">
@@
 <signal name="N$21">
 <contactref element="R211" pad="2"/>
-<contactref element="IC2" pad="4"/>
-<wire x1="29.49" y1="52.705" x2="27.305" y2="52.705" width="0.4064" layer="1"/>
 <wire x1="27.305" y1="52.705" x2="26.67" y2="53.34" width="0.4064" layer="1"/>
 <wire x1="26.67" y1="53.34" x2="26.67" y2="53.188" width="0.4064" layer="1"/>
+<contactref element="U$1" pad="2"/>
+<wire x1="27.305" y1="52.705" x2="28.575" y2="52.705" width="0.4064" layer="1"/>
+<wire x1="28.575" y1="52.705" x2="30.48" y2="54.61" width="0.4064" layer="1"/>
 </signal>
 <signal name="N$27">
 <contactref element="R210" pad="2"/>
-<contactref element="IC2" pad="5"/>
-<wire x1="29.49" y1="51.435" x2="27.305" y2="51.435" width="0.4064" layer="1"/>
 <wire x1="27.305" y1="51.435" x2="26.67" y2="50.8" width="0.4064" layer="1"/>
 <wire x1="26.67" y1="50.8" x2="26.67" y2="50.952" width="0.4064" layer="1"/>
+<contactref element="U$1" pad="3"/>
+<wire x1="27.305" y1="51.435" x2="29.845" y2="51.435" width="0.4064" layer="1"/>
+<wire x1="29.845" y1="51.435" x2="30.48" y2="52.07" width="0.4064" layer="1"/>
 </signal>
 <signal name="N$29">
@@
 <wire x1="60.808" y1="45.72" x2="60.808" y2="48.26" width="0.4064" layer="1"/>
 </signal>
-<signal name="N$14">
-<contactref element="R216" pad="1"/>
-<contactref element="IC2" pad="2"/>
-<wire x1="29.49" y1="55.245" x2="31.115" y2="55.245" width="0.4064" layer="1"/>
-<via x="31.115" y="55.245" extent="1-16" drill="0.5"/>
-<wire x1="31.115" y1="55.245" x2="32.868" y2="55.245" width="0.4064" layer="16"/>
-<wire x1="32.868" y1="55.245" x2="33.02" y2="55.397" width="0.4064" layer="16"/>
-</signal>
-<signal name="N$20">
-<contactref element="R217" pad="1"/>
-<contactref element="IC2" pad="15"/>
-<wire x1="39.09" y1="55.245" x2="37.465" y2="55.245" width="0.4064" layer="1"/>
-<via x="37.465" y="55.245" extent="1-16" drill="0.5"/>
-<wire x1="37.465" y1="55.245" x2="35.712" y2="55.245" width="0.4064" layer="16"/>
-<wire x1="35.712" y1="55.245" x2="35.56" y2="55.397" width="0.4064" layer="16"/>
-</signal>
 <signal name="N$5">
 <contactref element="C236" pad="2"/>
@@
 <wire x1="71.755" y1="48.743" x2="71.272" y2="48.26" width="0.4064" layer="1"/>
 </signal>
+<signal name="N$1">
+<contactref element="U$1" pad="1"/>
+<contactref element="R216" pad="1"/>
+<wire x1="30.48" y1="57.15" x2="31.267" y2="57.15" width="0.4064" layer="16"/>
+<wire x1="31.267" y1="57.15" x2="33.02" y2="55.397" width="0.4064" layer="16"/>
+</signal>
+<signal name="N$2">
+<contactref element="U$1" pad="8"/>
+<contactref element="R217" pad="1"/>
+<wire x1="38.1" y1="57.15" x2="37.313" y2="57.15" width="0.4064" layer="16"/>
+<wire x1="37.313" y1="57.15" x2="35.56" y2="55.397" width="0.4064" layer="16"/>
+</signal>
 </signals>
